Commit message: warehouse

File: src/amr_simulation/models/amr_waffle.sdf.xacro (robot description, xacro)
@@ -145,5 +145,5 @@
         </inertial>
         <collision name="wheel_left_collision">
-          <pose>0 0 0 -1.57 0 0</pose>
+          <pose>0 0 0 0 0 0</pose>
           <geometry>
             <cylinder>
@@ -158,6 +158,6 @@
                      longitudinal slip made command-integrated odom advance
                      while the physical model barely moved. -->
-                <mu>100</mu>
-                <mu2>100</mu2>
+                <mu>5.0</mu>
+                <mu2>1.5</mu2>
                 <slip1>0</slip1>
                 <slip2>0</slip2>
@@ -178,5 +178,5 @@
         </collision>
         <visual name="wheel_left_visual">
-          <pose>0 0 0 -1.57 0 0</pose>
+          <pose>0 0 0 0 0 0</pose>
           <geometry>
             <mesh>
@@ -214,6 +214,6 @@
             <friction>
               <ode>
-                <mu>100</mu>
-                <mu2>100</mu2>
+                <mu>5.0</mu>
+                <mu2>1.5</mu2>
                 <slip1>0</slip1>
                 <slip2>0</slip2>
@@ -266,4 +266,5 @@
           </geometry>
           <surface>
+            <friction><ode><mu>0.08</mu><mu2>0.08</mu2></ode></friction>
             <contact>
               <ode>
@@ -299,4 +300,5 @@
           </geometry>
           <surface>
+            <friction><ode><mu>0.08</mu><mu2>0.08</mu2></ode></friction>
             <contact>
               <ode>
@@ -386,9 +388,9 @@
         </axis>
       </joint>
-      <joint name='caster_back_right_joint' type='ball'>
+      <joint name='caster_back_right_joint' type='fixed'>
         <parent>base_link</parent>
         <child>caster_back_right_link</child>
       </joint>
-      <joint name='caster_back_left_joint' type='ball'>
+      <joint name='caster_back_left_joint' type='fixed'>
         <parent>base_link</parent>
         <child>caster_back_left_link</child>
